Commit message: update

File: robot/xarm.urdf (robot description, URDF)
Before this commit: robot xArm, 7 links, 6 joints
Links:
- added link gripper_base; visual box size=0.044 0.023 0.0285
- link base_link: geometry visual box size=0.16 0.16 0.01; visual cylinder length=0.012 radius=0.06
- link link5: geometry visual box size=0.044 0.023 0.0285; visual cylinder length=0.004 radius=0.01
Joints:
- removed joint arm1
- removed joint arm2
- removed joint arm3
- removed joint arm4
- removed joint arm5
- added joint base: type revolute, parent base_link, child link1, origin xyz=0.0 0.0 0.05 rpy=0.0 0.0 0.0, axis 0 0 1, limit lower=-3 upper=3 velocity=2.09
- added joint elbow: type revolute, parent link2, child link3, origin xyz=0.0 0.0 0.0965 rpy=0.0 0.0 0.0, axis 0 1 0, limit lower=-1.5708 upper=1.5708 velocity=2.09
- added joint shoulder: type revolute, parent link1, child link2, origin xyz=0.0 0.0 0.0425 rpy=0.0 0.0 0.0, axis 0 1 0, limit lower=-1.5708 upper=1.5708 velocity=2.09
- added joint wrist: type revolute, parent link3, child link4, origin xyz=0.0 0.0 0.0965 rpy=0.0 0.0 0.0, axis 0 1 0, limit lower=-1.5708 upper=1.5708 velocity=2.09
- added joint wristRotation: type revolute, parent link4, child link5, origin xyz=0.0 0.0 0.055 rpy=0.0 0.0 0.0, axis 0 0 1, limit lower=-1.5708 upper=1.5708 velocity=2.09
- joint world_joint: origin xyz=0.0 0.0 0.05 rpy=0.0 0.0 0.0 -> xyz=0.0 0.0 0.0 rpy=0.0 0.0 0.0

Commit message: update

File: robot/xarm.urdf (robot description, URDF)
Before this commit: robot xArm, 8 links, 6 joints
Links:
- removed link gripper_base
- link base_link: mass None -> 1
- link link1: mass None -> 1
- link link2: mass None -> 1
- link link3: mass None -> 1
- link link4: mass None -> 1
- link link5: mass None -> 1

Commit message: .

File: robot/xarm.urdf (robot description, URDF)
Before this commit: robot xArm, 7 links, 6 joints
Links:
- added link gripper_left_link, mass 1; visual cylinder length=0.05 radius=0.005
- added link gripper_right_link, mass 1; visual cylinder length=0.05 radius=0.005
Joints:
- added joint gripper_left: type revolute, parent link5, child gripper_left_link, origin xyz=0.0 0.02 0.01 rpy=0.0 0. 0.0, axis 1 0 0, limit lower=-1.5708 upper=1.5708 velocity=2.09
- added joint gripper_right: type revolute, parent link5, child gripper_right_link, origin xyz=0.0 -0.02 0.01 rpy=0.0 0.0 0.0, axis -1 0 0, limit lower=-1.5708 upper=1.5708 velocity=2.09
