Commit message: update name

File: src/assets/xarm.urdf (robot description, URDF)
Before this commit: robot xArm, 9 links, 8 joints
Joints:
- removed joint base
- removed joint elbow
- removed joint gripper_left
- removed joint gripper_right
- removed joint shoulder
- removed joint wrist
- removed joint wristRotation
- added joint base_joint: type revolute, parent base_link, child base_swivel_link, origin xyz=0.0 0.0 0.034 rpy=0.0 0.0 -1.5708, axis 0 0 1, limit lower=-3 upper=3 velocity=2.09
- added joint elbow_joint: type revolute, parent upperarm_link, child forearm_link, origin xyz=0.0 0.0 0.101 rpy=0.0 0.0 0.0, axis 1 0 0, limit lower=-1.5708 upper=1.5708 velocity=2.09
- added joint gripper_left_joint: type revolute, parent hand_link, child gripper_left_link, origin xyz=0.0 0.02 0.03 rpy=0.0 0. 0.0, axis -1 0 0, limit lower=-1.5708 upper=1.5708 velocity=2.09
- added joint gripper_right_joint: type revolute, parent hand_link, child gripper_right_link, origin xyz=0.0 -0.02 0.03 rpy=0.0 0.0 0.0, axis 1 0 0, limit lower=-1.5708 upper=1.5708 velocity=2.09
- added joint shoulder_joint: type revolute, parent base_swivel_link, child upperarm_link, origin xyz=0.0 0.0 0.031 rpy=0.0 0.0 0.0, axis 1 0 0, limit lower=-1.5708 upper=1.5708 velocity=2.09
- added joint wristRotation_joint: type revolute, parent wrist_link, child hand_link, origin xyz=0.0 0.0 0.055 rpy=0.0 0.0 1.5708, axis 0 0 1, limit lower=-1.5708 upper=1.5708 velocity=2.09
- added joint wrist_joint: type revolute, parent forearm_link, child wrist_link, origin xyz=0.0 0.0 0.0965 rpy=0.0 0.0 0.0, axis 1 0 0, limit lower=-1.5708 upper=1.5708 velocity=2.09
