Commit message: for the record

File: neu_ro_arm/assets/camera.urdf (robot description, URDF)
Before this commit: robot Camera, 4 links, 3 joints
Links:
- added link dummy_holder_link, mass 1
- link base_link: geometry collision box size=0.06 0.06 0.015; collision cylinder length=0.3048 radius=0.0047625
- link camera_link: geometry collision box size=0.04 0.03 0.04; visual mesh filename=src/assets/meshes/camera_with_holder.dae
- link holder_link: geometry collision box size=0.02 0.05 0.012; visual mesh filename=src/assets/meshes/top_rod_holder.dae
Joints:
- removed joint pitch_joint
- removed joint yaw_joint
- added joint height: type prismatic, parent dummy_holder_link, child base_link, origin xyz=0.0 0.0 0.0 rpy=0.0 0.0 0.0, axis 0 0 -1, limit lower=0.03 upper=0.3 velocity=1
- added joint pitch: type revolute, parent camera_link, child holder_link, origin xyz=0.0 0.027 0.0 rpy=0.0 0.0 0.0, axis 0 0 1, limit lower=0 upper=6.28319 velocity=1
- added joint yaw: type revolute, parent holder_link, child dummy_holder_link, origin xyz=0.0 0.0 0.0 rpy=0.0 0.0 0.0, axis 0 0 1, limit lower=0 upper=6.28319 velocity=1
- joint world_joint: child base_link -> camera_link
