Commit message: added docs

File: neu_ro_arm/assets/urdf/camera.urdf (robot description, URDF)
Before this commit: robot Camera, 2 links, 1 joints
Links:
- link camera_link: geometry collision box size=0.06 0.04 0.04; collision cylinder length=0.056 radius=0.016

File: neu_ro_arm/assets/urdf/camera_rod.urdf (robot description, URDF)
Before this commit: robot Rod, 2 links, 1 joints
Links:
- link rod_link: geometry collision cylinder length=0.3 radius=0.01; visual cylinder length=0.3 radius=0.005

File: neu_ro_arm/assets/urdf/xarm.urdf (robot description, URDF)
Before this commit: robot xArm, 9 links, 8 joints
Links:
- link base_link: geometry collision box size=0.154 0.14 0.04; visual mesh filename=assets/meshes/base.dae
- link base_swivel_link: geometry collision cylinder length=0.04 radius=0.06; visual mesh filename=assets/meshes/base_swivel.dae
- link forearm_link: geometry collision box size=0.05 0.04 0.11; visual mesh filename=assets/meshes/forearm_link.dae
- link gripper_left_link: geometry collision cylinder length=0.06 radius=0.005; visual cylinder length=0.06 radius=0.005
- link gripper_right_link: geometry collision cylinder length=0.06 radius=0.005; visual cylinder length=0.06 radius=0.005
- link upperarm_link: geometry collision box size=0.055 0.04 0.11; visual mesh filename=assets/meshes/upperarm_link.dae
- link wrist_link: geometry collision box size=0.05 0.04 0.06; visual mesh filename=assets/meshes/lx15d_double.dae

Commit message: urdf mesh path changed to absolute

File: neu_ro_arm/assets/urdf/camera.urdf (robot description, URDF)
Before this commit: robot Camera, 2 links, 1 joints
Links:
- link camera_link: geometry collision box size=0.06 0.04 0.04; collision cylinder length=0.056 radius=0.016

File: neu_ro_arm/assets/urdf/xarm.urdf (robot description, URDF)
Before this commit: robot xArm, 9 links, 8 joints
Links:
- link base_link: geometry collision box size=0.154 0.14 0.04; visual mesh filename=neu_ro_arm/assets/meshes/base.dae
- link base_swivel_link: geometry collision cylinder length=0.04 radius=0.06; visual mesh filename=neu_ro_arm/assets/meshes/base_swivel.dae
- link forearm_link: geometry collision box size=0.05 0.04 0.11; visual mesh filename=neu_ro_arm/assets/meshes/forearm_link.dae
- link upperarm_link: geometry collision box size=0.055 0.04 0.11; visual mesh filename=neu_ro_arm/assets/meshes/upperarm_link.dae
- link wrist_link: geometry collision box size=0.05 0.04 0.06; visual mesh filename=neu_ro_arm/assets/meshes/lx15d_double.dae
