Commit message: removed collision at bottom so theres no contact with robotbase

File: neu_ro_arm/assets/urdf/camera_rod.urdf (robot description, URDF)
Before this commit: robot Rod, 2 links, 1 joints
Links:
- link rod_link: geometry collision cylinder length=0.25 radius=0.01; visual cylinder length=0.25 radius=0.005

Commit message: adjusted collision parameters so robot base didnt intersect camera rod

File: neu_ro_arm/assets/urdf/camera_rod.urdf (robot description, URDF)
Before this commit: robot Rod, 2 links, 1 joints
Links:
- link rod_link: geometry collision cylinder length=0.2048 radius=0.01; visual cylinder length=0.3048 radius=0.005

File: neu_ro_arm/assets/urdf/xarm.urdf (robot description, URDF)
Before this commit: robot xArm, 10 links, 9 joints
Links:
- link base_link: geometry collision box size=0.154 0.14 0.005; visual mesh filename=neu_ro_arm/assets/meshes/base.dae
- link base_swivel_link: geometry collision cylinder length=0.04 radius=0.075; visual mesh filename=neu_ro_arm/assets/meshes/base_swivel.dae
Joints:
- joint gripper_left_joint: limit lower=1e-4 upper=0.04243 velocity=0.001 -> lower=5e-4 upper=0.04243 velocity=0.001
- joint gripper_right_joint: limit lower=1e-4 upper=0.04243 velocity=0.001 -> lower=5e-4 upper=0.04243 velocity=0.001
