Commit message: update

File: neu_ro_arm/assets/urdf/xarm.urdf (robot description, URDF)
Before this commit: robot xArm, 9 links, 8 joints
Joints:
- joint elbow_joint: axis 1 0 0 -> -1 0 0
- joint shoulder_joint: axis 1 0 0 -> -1 0 0

Commit message: changed gripper to prismatic

File: neu_ro_arm/assets/urdf/xarm.urdf (robot description, URDF)
Before this commit: robot xArm, 9 links, 8 joints
Links:
- added link virtual_palm_link, mass 1; visual sphere radius=0.005
- link gripper_left_link: geometry collision box size=0.02 0.008 0.06; visual box size=0.02 0.008 0.06
- link gripper_right_link: geometry collision box size=0.02 0.008 0.06; visual box size=0.02 0.008 0.06
- link hand_link: geometry collision box size=0.044 0.023 0.0285; visual box size=0.04 0.04 0.02
Joints:
- added joint virtual_palm_joint: type fixed, parent hand_link, child virtual_palm_link, origin xyz=0.0 0.0 0.110 rpy=0.0 0.0 0.0
- joint gripper_left_joint: axis -1 0 0 -> 1 0 -1; limit lower=-1.5708 upper=1.5708 velocity=2.09 -> lower=0 upper=0.04243 velocity=0.1; origin xyz=0.0 0.02 0.03 rpy=0.0 0. 0.0 -> xyz=0.014 0.0 0.062 rpy=0.0 0. 0.0; type revolute -> prismatic
- joint gripper_right_joint: axis 1 0 0 -> -1 0 -1; limit lower=-1.5708 upper=1.5708 velocity=2.09 -> lower=0 upper=0.04243 velocity=0.1; origin xyz=0.0 -0.02 0.03 rpy=0.0 0.0 0.0 -> xyz=-0.014 0.0 0.062 rpy=0.0 0.0 0.0; type revolute -> prismatic
- joint wristRotation_joint: origin xyz=0.0 0.0 0.055 rpy=0.0 0.0 1.5708 -> xyz=0.0 0.0 0.052 rpy=0.0 0.0 0
- joint wrist_joint: axis 1 0 0 -> -1 0 0

Commit message: added virtual palm end effector link; included damping on joints

File: neu_ro_arm/assets/urdf/xarm.urdf (robot description, URDF)
Before this commit: robot xArm, 10 links, 9 joints
Joints:
- joint gripper_left_joint: limit lower=0 upper=0.04243 velocity=0.1 -> lower=1e-4 upper=0.04243 velocity=0.001
- joint gripper_right_joint: limit lower=0 upper=0.04243 velocity=0.1 -> lower=1e-4 upper=0.04243 velocity=0.001

Commit message: padded collisions of arm

File: neu_ro_arm/assets/urdf/xarm.urdf (robot description, URDF)
Before this commit: robot xArm, 10 links, 9 joints
Links:
- link base_link: geometry collision box size=0.154 0.14 0.05; visual mesh filename=neu_ro_arm/assets/meshes/base.dae
- link base_swivel_link: geometry collision cylinder length=0.04 radius=0.08; visual mesh filename=neu_ro_arm/assets/meshes/base_swivel.dae
- link forearm_link: geometry collision box size=0.05 0.05 0.11; visual mesh filename=neu_ro_arm/assets/meshes/forearm_link.dae
- link hand_link: geometry collision box size=0.06 0.05 0.05; visual box size=0.04 0.04 0.02
- link upperarm_link: geometry collision box size=0.06 0.04 0.11; visual mesh filename=neu_ro_arm/assets/meshes/upperarm_link.dae
- link wrist_link: geometry collision box size=0.05 0.055 0.06; visual mesh filename=neu_ro_arm/assets/meshes/lx15d_double.dae

Commit message: fixed prismatic joint axis so warning is not given

File: neu_ro_arm/assets/urdf/xarm.urdf (robot description, URDF)
Before this commit: robot xArm, 10 links, 9 joints
Joints:
- joint gripper_left_joint: axis 1 0 -1 -> 0.7071067811865476 0 -0.7071067811865476
- joint gripper_right_joint: axis -1 0 -1 -> -0.7071067811865476 0 -0.7071067811865476

Commit message: adjusted joint limits to reflect xArm's

File: neu_ro_arm/assets/urdf/xarm.urdf (robot description, URDF)
Before this commit: robot xArm, 10 links, 9 joints
Joints:
- joint base_joint: limit lower=-3 upper=3 velocity=2.09 -> lower=-2.0 upper=2.0 velocity=2.09
- joint elbow_joint: limit lower=-1.5708 upper=1.5708 velocity=2.09 -> lower=-2.0 upper=2.0 velocity=2.09
- joint shoulder_joint: limit lower=-1.5708 upper=1.5708 velocity=2.09 -> lower=-2.0 upper=2.0 velocity=2.09
- joint wristRotation_joint: limit lower=-1.5708 upper=1.5708 velocity=2.09 -> lower=-2.0 upper=2.0 velocity=2.09
- joint wrist_joint: limit lower=-1.5708 upper=1.5708 velocity=2.09 -> lower=-2.0 upper=2.0 velocity=2.09

Commit message: more accurate gripper mechanism

File: neu_ro_arm/assets/urdf/xarm.urdf (robot description, URDF)
Before this commit: robot xArm, 10 links, 9 joints
Links:
- removed link base_swivel_link
- removed link gripper_left_link
- removed link gripper_right_link
- removed link virtual_palm_link
- added link left_finger_bar_link, mass 0.01; collision box size=0.018 0.003 0.003; visual mesh filename=neu_ro_arm/assets/meshes/left_finger_bar.dae scale=10.0 1.0 1.0
- added link left_finger_base_link, mass 0.01; collision box size=0.01 0.0375 0.003; visual mesh filename=neu_ro_arm/assets/meshes/right_finger_base.dae scale=1.0 1.0 1.0
- added link left_finger_tip_link, mass 0.01; collision mesh filename=neu_ro_arm/assets/meshes/Circle.002.dae scale=1.0 1.0 1.0; visual mesh filename=neu_ro_arm/assets/meshes/left_finger_tip.dae scale=1.0 1.0 1.0
- added link right_finger_bar_link, mass 0.01; collision box size=0.018 0.003 0.003; visual mesh filename=neu_ro_arm/assets/meshes/right_finger_bar.dae scale=10.0 1.0 1.0
- added link right_finger_base_link, mass 0.01; collision box size=0.01 0.0375 0.003; visual mesh filename=neu_ro_arm/assets/meshes/right_finger_base.dae scale=1.0 1.0 1.0
- added link right_finger_tip_link, mass 0.01; collision mesh filename=neu_ro_arm/assets/meshes/Circle.003.dae scale=1.0 1.0 1.0; visual mesh filename=neu_ro_arm/assets/meshes/right_finger_tip.dae scale=1.0 1.0 1.0
- added link swivel_link, mass 0.15; collision box size=0.04350001 0.0400 0.02775; visual mesh filename=neu_ro_arm/assets/meshes/shoulder_servo.dae scale=20.0 20.0 10.0
- added link virtual_grasp_link, mass 0.001; visual sphere radius=0.003
- link base_link: mass 1 -> 0.15; geometry collision box size=0.07606218 0.0770 0.0320; collision box size=0.15400229 0.1400 0.0020
- link forearm_link: mass 1 -> 0.04; geometry collision box size=0.0230 0.09 0.03512; visual mesh filename=neu_ro_arm/assets/meshes/forearm_lower_servo.dae scale=11.5 22.00001 13.5
- link hand_link: mass 1 -> 0.02; geometry collision box size=0.0230 0.0440 0.03106; collision cylinder length=0.00451872 radius=0.03339804
- link upperarm_link: mass 1 -> 0.1; geometry collision box size=0.05600002 0.0320 0.11; visual mesh filename=neu_ro_arm/assets/meshes/upperarm_lower.dae scale=1.0 1.0 1.0
- link wrist_link: mass 1 -> 0.02; geometry collision box size=0.0470 0.0405 0.06475; visual mesh filename=neu_ro_arm/assets/meshes/wrist_metal_part.dae scale=1.0 1.0 1.0
Joints:
- removed joint gripper_left_joint
- removed joint gripper_right_joint
- removed joint virtual_palm_joint
- removed joint wristRotation_joint
- added joint left_finger_joint: type revolute, parent left_finger_base_link, child left_finger_tip_link, origin xyz=0.00002379 0.03001281 -0.0075 rpy=0 0 0.44359, axis 0 0 -1.0, limit lower=-2.0 upper=2.0 velocity=2.0
- added joint left_finger_linkage_joint: type revolute, parent hand_link, child left_finger_bar_link, origin xyz=0.0045 -0.00852974 0.01950001 rpy=1.5708 -1.5708 0, axis 0 0 -1.0, limit lower=0.0 upper=1.5 effort=0 velocity=2.0
- added joint left_knuckle_joint: type revolute, parent hand_link, child left_finger_base_link, origin xyz=0.014 -0.006 0 rpy=1.5708 0 0, axis 0 0 -1.0, limit lower=0.05 upper=1.38 effort=0 velocity=2.0
- added joint right_finger_joint: type revolute, parent right_finger_base_link, child right_finger_tip_link, origin xyz=-0.00002379 0.03001281 -0.0015 rpy=0 0 2.01439, axis 0 0 1.0, limit lower=-2.0 upper=2.0 effort=0 velocity=2.0
- added joint right_finger_linkage_joint: type revolute, parent hand_link, child right_finger_bar_link, origin xyz=-0.0045 -0.00852974 0.01950001 rpy=1.5708 1.5708 0, axis 0 0 1.0, limit lower=0.0 upper=1.5 effort=0 velocity=2.0
- added joint right_knuckle_joint: type revolute, parent hand_link, child right_finger_base_link, origin xyz=-0.0140 -0.006 0 rpy=1.5708 0 0, axis 0 0 1.0, limit lower=0.05 upper=1.38 effort=0 velocity=2.0
- added joint virtual_grasp_joint: type fixed, parent hand_link, child virtual_grasp_link, origin xyz=0.0 0.0 0.076 rpy=0.0 0.0 0.0
- added joint wrist_rotation_joint: type revolute, parent wrist_link, child hand_link, origin xyz=0 -0.08378503 0 rpy=1.5708 -1.5708 0, axis 0 0 1.0, limit lower=-2.0 upper=2.0 effort=0 velocity=2.0
- joint base_joint: axis 0 0 1 -> 0 0 1.0; child base_swivel_link -> swivel_link; limit lower=-2.0 upper=2.0 velocity=2.09 -> lower=-2.0 upper=2.0 effort=0 velocity=2.0; origin xyz=0.0 0.0 0.034 rpy=0.0 0.0 -1.5708 -> xyz=0 0 0.03953818 rpy=0 0 1.5708
- joint elbow_joint: axis -1 0 0 -> 0 0 1.0; limit lower=-2.0 upper=2.0 velocity=2.09 -> lower=-2.0 upper=2.0 effort=0 velocity=2.0; origin xyz=0.0 0.0 0.101 rpy=0.0 0.0 0.0 -> xyz=-0.09883501 0 0 rpy=0 0 1.5708
- joint shoulder_joint: axis -1 0 0 -> 0 0 1.0; limit lower=-2.0 upper=2.0 velocity=2.09 -> lower=-1.58 upper=1.58 effort=0 velocity=2.0; origin xyz=0.0 0.0 0.031 rpy=0.0 0.0 0.0 -> xyz=0 0 0.024195 rpy=0 1.5708 0; parent base_swivel_link -> swivel_link
- joint world_joint: origin xyz=0.0 0.0 0.012 rpy=0.0 0.0 1.5708 -> xyz=0.0 0.0 0.012 rpy=0.0 0.0 0.0
- joint wrist_joint: axis -1 0 0 -> 0 0 1.0; limit lower=-2.0 upper=2.0 velocity=2.09 -> lower=-2.0 upper=2.0 effort=0 velocity=2.0; origin xyz=0.0 0.0 0.0965 rpy=0.0 0.0 0.0 -> xyz=0 0.09468611 0 rpy=0 0 3.14159

Commit message: fixed instabilities with gripper

File: neu_ro_arm/assets/urdf/xarm.urdf (robot description, URDF)
Before this commit: robot xarm, 14 links, 13 joints
Links:
- link hand_link: geometry collision box size=0.0230 0.0440 0.03106; collision cylinder length=0.00451872 radius=0.025
- link left_finger_bar_link: geometry collision box size=0.012 0.003 0.003; visual mesh filename=neu_ro_arm/assets/meshes/left_finger_bar.dae scale=10.0 1.0 1.0
- link left_finger_tip_link: geometry collision mesh filename=neu_ro_arm/assets/meshes/left_finger_tip.dae scale=1.0 1.0 1.0; visual mesh filename=neu_ro_arm/assets/meshes/left_finger_tip.dae scale=1.0 1.0 1.0
- link right_finger_bar_link: geometry collision box size=0.012 0.003 0.003; visual mesh filename=neu_ro_arm/assets/meshes/left_finger_bar.dae scale=10.0 1.0 1.0
- link right_finger_tip_link: geometry collision mesh filename=neu_ro_arm/assets/meshes/left_finger_tip.dae scale=1.0 1.0 1.0; visual mesh filename=neu_ro_arm/assets/meshes/left_finger_tip.dae scale=1.0 1.0 1.0
Joints:
- joint elbow_joint: limit lower=-2.0 upper=2.0 effort=0 velocity=2.0 -> lower=-2.0 upper=2.0 velocity=2.0
- joint left_finger_joint: origin xyz=0.00002379 0.03001281 -0.0075 rpy=0 0 0.44359 -> xyz=0.00 0.03 -0.0 rpy=0 0 0.0
- joint left_finger_linkage_joint: axis 0 0 -1.0 -> 0 -1 0; limit lower=0.0 upper=1.5 effort=0 velocity=2.0 -> lower=0.0 upper=1.5 velocity=2.0; origin xyz=0.0045 -0.00852974 0.01950001 rpy=1.5708 -1.5708 0 -> xyz=0.0045 0 0.0195 rpy=0 0 0
- joint left_knuckle_joint: limit lower=0.05 upper=1.38 effort=0 velocity=2.0 -> lower=0.05 upper=1.6 velocity=2.0; origin xyz=0.014 -0.006 0 rpy=1.5708 0 0 -> xyz=0.014 0.0 0 rpy=1.5708 0 0
- joint right_finger_joint: origin xyz=-0.00002379 0.03001281 -0.0015 rpy=0 0 2.01439 -> xyz=0.0 0.03 0 rpy=0 0 0
- joint right_finger_linkage_joint: axis 0 0 1.0 -> 0 1 0; limit lower=0.0 upper=1.5 effort=0 velocity=2.0 -> lower=0 upper=1.5 effort=0 velocity=2.0; origin xyz=-0.0045 -0.00852974 0.01950001 rpy=1.5708 1.5708 0 -> xyz=-0.0045 0.0 0.0195 rpy=0 0 0
- joint right_knuckle_joint: limit lower=0.05 upper=1.38 effort=0 velocity=2.0 -> lower=0.05 upper=1.6 effort=0 velocity=2.0; origin xyz=-0.0140 -0.006 0 rpy=1.5708 0 0 -> xyz=-0.014 0 0 rpy=1.5708 0 0
- joint wrist_joint: limit lower=-2.0 upper=2.0 effort=0 velocity=2.0 -> lower=-1.8 upper=2.0 velocity=2.0
- joint wrist_rotation_joint: limit lower=-2.0 upper=2.0 effort=0 velocity=2.0 -> lower=-2.0 upper=2.0 velocity=2.0

Commit message: fixed end effector pose setting

File: neu_ro_arm/assets/urdf/xarm.urdf (robot description, URDF)
Before this commit: robot xarm, 14 links, 13 joints
Links:
- link left_finger_bar_link: geometry collision box size=0.003 0.003 0.003; visual mesh filename=neu_ro_arm/assets/meshes/left_finger_bar.dae scale=10.0 1.0 1.0
- link right_finger_bar_link: geometry collision box size=0.003 0.003 0.003; visual mesh filename=neu_ro_arm/assets/meshes/left_finger_bar.dae scale=10.0 1.0 1.0

Commit message: refactored pybullet simulator so it can be used by controller and motion planner concurrently

File: neu_ro_arm/assets/urdf/xarm.urdf (robot description, URDF)
Before this commit: robot xarm, 14 links, 13 joints
Joints:
- joint world_joint: origin xyz=0.0 0.0 0.012 rpy=0.0 0.0 0.0 -> xyz=0.0 0.0 0.0 rpy=0.0 0.0 0.0

Commit message: switched to stl for xarm urdf

File: neu_ro_arm/assets/urdf/xarm.urdf (robot description, URDF)
Before this commit: robot xarm, 14 links, 13 joints
Links:
- removed link left_finger_bar_link
- removed link right_finger_bar_link
- added link dummy_link, mass 0.01
- link base_link: geometry collision box size=0.07606218 0.0770 0.0320; collision box size=0.15400229 0.1400 0.0020
- link forearm_link: geometry collision box size=0.023 0.035 0.09; visual mesh filename=neu_ro_arm/assets/meshes/forearm.stl scale=0.001 0.001 0.001
- link hand_link: geometry collision cylinder length=0.00451872 radius=0.025; visual mesh filename=neu_ro_arm/assets/meshes/hand.stl scale=0.001 0.001 0.001
- link left_finger_base_link: mass 0.01 -> 0.1; geometry collision box size=0.003 0.01 0.0375; visual mesh filename=neu_ro_arm/assets/meshes/finger_base.stl scale=0.001 0.001 0.001
- link left_finger_tip_link: geometry collision box size=0.008 0.008 0.012; visual mesh filename=neu_ro_arm/assets/meshes/finger_tip.stl scale=0.001 0.001 0.001
- link right_finger_base_link: mass 0.01 -> 0.1; geometry collision box size=0.003 0.01 0.0375; visual mesh filename=neu_ro_arm/assets/meshes/finger_base.stl scale=0.001 0.001 0.001
- link right_finger_tip_link: geometry collision box size=0.008 0.008 0.012; visual mesh filename=neu_ro_arm/assets/meshes/finger_tip.stl scale=0.001 0.001 0.001
- link swivel_link: geometry collision box size=0.04350001 0.0400 0.02775; visual mesh filename=neu_ro_arm/assets/meshes/swivel.stl scale=0.001 0.001 0.001
- link upperarm_link: geometry collision box size=0.032 0.056 0.11; visual mesh filename=neu_ro_arm/assets/meshes/upperarm.stl scale=0.001 0.001 0.001
- link wrist_link: geometry collision box size=0.045 0.047 0.06475; visual mesh filename=neu_ro_arm/assets/meshes/wrist.stl scale=0.001 0.001 0.001
Joints:
- removed joint left_finger_joint
- removed joint left_finger_linkage_joint
- removed joint right_finger_joint
- removed joint right_finger_linkage_joint
- added joint dummy_y_joint: type prismatic, parent dummy_link, child left_finger_tip_link, origin xyz=0.0 0.0 0.0 rpy=0.0 0.0 0.0, axis 0 1 0, limit lower=0.0145 upper=0.0445 effort=1000 velocity=2.0
- added joint dummy_z_joint: type prismatic, parent hand_link, child dummy_link, origin xyz=0.0 0.0 0.0 rpy=0.0 0.0 0.0, axis 0 0 1, limit lower=0.025 upper=0.055 effort=1000 velocity=2.0
- added joint finger_separation_joint: type prismatic, parent left_finger_tip_link, child right_finger_tip_link, origin xyz=0.0 0.00 0.0 rpy=0.0 0.0 0.0, axis 0 -1 0, limit lower=0.029 upper=0.089 effort=1000 velocity=2.0
- joint base_joint: origin xyz=0 0 0.03953818 rpy=0 0 1.5708 -> xyz=0 0 0.047 rpy=0 0 0
- joint elbow_joint: axis 0 0 1.0 -> 0 1 0; origin xyz=-0.09883501 0 0 rpy=0 0 1.5708 -> xyz=0 0 0.0988 rpy=0 0 0
- joint left_knuckle_joint: axis 0 0 -1.0 -> -1 0 0; limit lower=0.05 upper=1.6 velocity=2.0 -> lower=0.05 upper=1.6 effort=1000 velocity=2.0; origin xyz=0.014 0.0 0 rpy=1.5708 0 0 -> xyz=0 0.014 0.025 rpy=0 0 0
- joint right_knuckle_joint: axis 0 0 1.0 -> 1 0 0; limit lower=0.05 upper=1.6 effort=0 velocity=2.0 -> lower=0.05 upper=1.6 effort=1000 velocity=2.0; origin xyz=-0.014 0 0 rpy=1.5708 0 0 -> xyz=0 -0.014 0.025 rpy=0 0 0
- joint shoulder_joint: axis 0 0 1.0 -> 0 1 0; origin xyz=0 0 0.024195 rpy=0 1.5708 0 -> xyz=0 0 0.0177 rpy=0 0 0
- joint virtual_grasp_joint: origin xyz=0.0 0.0 0.076 rpy=0.0 0.0 0.0 -> xyz=0.0 0.0 0.1 rpy=0.0 0.0 0.0
- joint wrist_joint: axis 0 0 1.0 -> 0 1 0; origin xyz=0 0.09468611 0 rpy=0 0 3.14159 -> xyz=0 0 0.0947 rpy=0 0 0
- joint wrist_rotation_joint: axis 0 0 1.0 -> 0 0 1; origin xyz=0 -0.08378503 0 rpy=1.5708 -1.5708 0 -> xyz=0 0 0.0588 rpy=0 0 0
