Commit message: typo in urdf; bug in gripper state calcualtion

File: nuro_arm/assets/urdf/xarm.urdf (robot description, URDF)
Before this commit: robot xarm, 13 links, 12 joints
Links:
- link base_link: geometry collision box size=0.07606218 0.0770 0.0320; collision box size=0.15400229 0.1400 0.0020
- link forearm_link: geometry collision box size=0.023 0.035 0.09; visual mesh filename=nuro_arm/assets/meshes/forearm.stl scale=0.001 0.001 0.001
- link hand_link: geometry collision cylinder length=0.00451872 radius=0.025; visual mesh filename=nuro_arm/assets/meshes/hand.stl scale=0.001 0.001 0.001
- link left_finger_base_link: geometry collision box size=0.003 0.01 0.0375; visual mesh filename=nuro_arm/assets/meshes/finger_base.stl scale=0.001 0.001 0.001
- link left_finger_tip_link: geometry collision box size=0.008 0.008 0.012; visual mesh filename=nuro_arm/assets/meshes/finger_tip.stl scale=0.001 0.001 0.001
- link right_finger_base_link: geometry collision box size=0.003 0.01 0.0375; visual mesh filename=nuro_arm/assets/meshes/finger_base.stl scale=0.001 0.001 0.001
- link right_finger_tip_link: geometry collision box size=0.008 0.008 0.012; visual mesh filename=nuro_arm/assets/meshes/finger_tip.stl scale=0.001 0.001 0.001
- link swivel_link: geometry collision box size=0.04350001 0.0400 0.02775; visual mesh filename=nuro_arm/assets/meshes/swivel.stl scale=0.001 0.001 0.001
- link upperarm_link: geometry collision box size=0.032 0.056 0.11; visual mesh filename=nuro_arm/assets/meshes/upperarm.stl scale=0.001 0.001 0.001
- link wrist_link: geometry collision box size=0.045 0.047 0.06475; visual mesh filename=nuro_arm/assets/meshes/wrist.stl scale=0.001 0.001 0.001

Commit message: added motor controlelr to urdf

File: nuro_arm/assets/urdf/xarm.urdf (robot description, URDF)
Before this commit: robot xarm, 13 links, 12 joints
Links:
- link base_link: geometry collision box size=0.07606218 0.0770 0.0320; collision box size=0.15400229 0.1400 0.0020
