Commit message: cleaning up:

File: nuro_arm/assets/urdf/camera.urdf (robot description, URDF)
Before this commit: robot Camera, 2 links, 1 joints
Links:
- link camera_link: geometry collision box size=0.06 0.04 0.04; collision cylinder length=0.056 radius=0.016

File: nuro_arm/assets/urdf/xarm.urdf (robot description, URDF)
Before this commit: robot xarm, 13 links, 12 joints
Links:
- link hand_link: geometry collision box size=0.03 0.04 0.02; collision cylinder length=0.00451872 radius=0.025
